File: kicad/fireplace/fireplace.sch (KiCad schematic (older format))
At the start: 18 parts, among them SW1 SW_Push, SW2 SW_Push, SW3 SW_Push, SW4 SW_Push, U1 ULN2003A, U2 PIC16F84-XX/P, U3 MOC3021M, U4 ATMEGA8-16AU, U5 QSE159, Y1 4MHz

Commit message: 1
Parts:
- added C?: 1u, symbol C
- added R?: 10k, symbol R
Connections:
- net labels added: LED_COM
- wire segments 67 -> 87
Other:
- moved on the sheet: U4, Y1
